Commit message: feat: :memo: Task1 Adding a RGB Camera

File: arduinobot_ws/src/arduinobot_description/urdf/arduinobot.urdf.xacro (robot description, xacro)
@@ -108,3 +108,17 @@
         <mimic joint="joint_4" multiplier="-1"/>
     </joint>
+    <link name="rgb_camera">
+        <visual>
+            <origin rpy="-${PI/2} 0 -${PI/2}" xyz="-0.07 0.12 0.12" />
+            <geometry>
+                <mesh filename="package://arduinobot_description/meshes/pi_camera.STL" scale="0.01 0.01 0.01"/>
+            </geometry>
+        </visual>
+    </link>
+    <joint name="rgb_camera_joint" type="fixed">
+        <parent link="base_link" />
+        <child link="rgb_camera" />
+        <axis xyz="0 0 0"/>
+        <origin rpy="0 -0.5 1.57" xyz="0 0.45 0.2"/>
+    </joint>
 </robot>

Commit message: perf: :construction_worker: Improved version of the URDF file

File: arduinobot_ws/src/arduinobot_description/urdf/arduinobot.urdf.xacro (robot description, xacro)
@@ -1,124 +1,190 @@
 <?xml version="1.0"?>
 <robot xmlns:xacro="http://www.ros.org/wiki/xacro" name="arduinobot">
-    <xacro:property name="PI" value="3.14159" />
+    <!-- Useful XACRO Variables (Properties) -->
+    <xacro:property name="PI" value="3.14159265359" />
     <xacro:property name="effort" value="30.0" />
     <xacro:property name="velocity" value="10.0" />
+    <!-- Useful Macros -->
+    <xacro:macro name="default_inertial" params="mass">
+        <inertial>
+            <origin xyz="0 0 0" rpy="0 0 0"/>
+            <mass value="${mass}" />
+            <inertia ixx="1.0" ixy="0.0" ixz="0.0"
+                     iyy="1.0" iyz="0.0"
+                     izz="1.0" />
+        </inertial>
+    </xacro:macro>
+    <!-- Links -->
     <link name="world"/>
-    <link name= "base_link">
+    <link name="base_link">
+        <xacro:default_inertial mass="1.0"/>
         <visual>
-            <origin rpy="0 0 0" xyz="-0.5 -0.5 0"/>
+            <origin xyz="-0.5 -0.5 0" rpy="0 0 0"/>
             <geometry>
                 <mesh filename="package://arduinobot_description/meshes/basement.STL" scale="0.01 0.01 0.01"/>
             </geometry>
         </visual>
+        <collision>
+            <origin xyz="-0.5 -0.5 0" rpy="0 0 0"/>
+            <geometry>
+                <mesh filename="package://arduinobot_description/meshes/basement.STL" scale="0.01 0.01 0.01"/>
+            </geometry>
+        </collision>
     </link>
-    <joint name="virtual_joint" type="fixed">
-        <parent link="world" />
-        <child link="base_link" />
-        <origin rpy="0 0 0" xyz="0 0 0" />
-    </joint>
     <link name="base_plate">
+        <xacro:default_inertial mass="0.1"/>
         <visual>
-                <origin rpy="0 0 0" xyz="-0.39 -0.39 -0.56"/>
+            <origin xyz="-0.39 -0.39 -0.56" rpy="0 0 0"/>
             <geometry>
                 <mesh filename="package://arduinobot_description/meshes/base_plate.STL" scale="0.01 0.01 0.01"/>
             </geometry>
         </visual>
+        <collision>
+            <origin xyz="-0.39 -0.39 -0.56" rpy="0 0 0"/>
+            <geometry>
+                <mesh filename="package://arduinobot_description/meshes/base_plate.STL" scale="0.01 0.01 0.01"/>
+            </geometry>
+        </collision>
     </link>
-    <joint name="joint_1" type="revolute">
-        <parent link="base_link" />
-        <child link="base_plate" />
-        <axis xyz="0 0 1"/>
-        <origin rpy="0 0 0" xyz="0 0 0.307" />
-        <limit lower="-${PI/2}" upper="${PI/2}" effort="${effort}" velocity="${velocity}"/>
-    </joint>
     <link name="forward_drive_arm">
+        <xacro:default_inertial mass="0.1"/>
         <visual>
-                <origin rpy="0 -${PI/2} ${PI/2}" xyz="0.19 0.06 -0.08"/>
+            <origin xyz="0.19 0.06 -0.08" rpy=" 0 -${PI/2} ${PI/2}"/>
             <geometry>
                 <mesh filename="package://arduinobot_description/meshes/forward_drive_arm.STL" scale="0.01 0.01 0.01"/>
             </geometry>
         </visual>
+        <collision>
+            <origin xyz="0.19 0.06 -0.08" rpy=" 0 -${PI/2} ${PI/2}"/>
+            <geometry>
+                <mesh filename="package://arduinobot_description/meshes/forward_drive_arm.STL" scale="0.01 0.01 0.01"/>
+            </geometry>
+        </collision>
     </link>
-    <joint name="joint_2" type="revolute">
-        <parent link="base_plate" />
-        <child link="forward_drive_arm" />
-        <axis xyz="1 0 0"/>
-        <origin rpy="0 0 0" xyz="-0.02 0 0.35" />
-        <limit lower="-${PI/2}" upper="${PI/2}" effort="${effort}" velocity="${velocity}"/>
-    </joint>
     <link name="horizontal_arm">
+        <xacro:default_inertial mass="0.1"/>
         <visual>
-                <origin rpy="${PI/2} 0 ${PI/2}" xyz="-0.03 -0.4 -0.06"/>
+            <origin xyz="-0.03 -0.4 -0.06" rpy="${PI/2} 0 ${PI/2}"/>
             <geometry>
                 <mesh filename="package://arduinobot_description/meshes/horizontal_arm.STL" scale="0.01 0.01 0.01"/>
             </geometry>
         </visual>
+        <collision>
+            <origin xyz="-0.03 -0.4 -0.06" rpy="${PI/2} 0 ${PI/2}"/>
+            <geometry>
+                <mesh filename="package://arduinobot_description/meshes/horizontal_arm.STL" scale="0.01 0.01 0.01"/>
+            </geometry>
+        </collision>
     </link>
-    <joint name="joint_3" type="revolute">
-        <parent link="forward_drive_arm" />
-        <child link="horizontal_arm" />
-        <axis xyz="1 0 0"/>
-        <origin rpy="0 0 0" xyz="0 0 0.8" />
-        <limit lower="-${PI/2}" upper="${PI/2}" effort="${effort}" velocity="${velocity}"/>
-    </joint>
     <link name="claw_support">
+        <xacro:default_inertial mass="0.05"/>
         <visual>
-                <origin rpy="0 0 ${PI/2}" xyz="0 -0.05 -0.15"/>
+            <origin xyz="0 -0.05 -0.15" rpy="0 0 ${PI/2}"/>
             <geometry>
                 <mesh filename="package://arduinobot_description/meshes/claw_support.STL" scale="0.01 0.01 0.01"/>
             </geometry>
         </visual>
+        <collision>
+            <origin xyz="0 -0.05 -0.15" rpy="0 0 ${PI/2}"/>
+            <geometry>
+                <mesh filename="package://arduinobot_description/meshes/claw_support.STL" scale="0.01 0.01 0.01"/>
+            </geometry>
+        </collision>
     </link>
-    <joint name="horizontal_arm_to_claw_support" type="fixed">
-        <parent link="horizontal_arm" />
-        <child link="claw_support" />
-        <axis xyz="1 0 0"/>
-        <origin rpy="0 0 0" xyz="0 0.82 0" />
-    </joint>
     <link name="gripper_right">
+        <xacro:default_inertial mass="0.01"/>
         <visual>
-                <origin rpy="0 0 -${PI/2}" xyz="-0.1 0.5 -0.1"/>
+            <origin xyz="-0.1 0.50 -0.1" rpy="0 0 -${PI/2}"/>
             <geometry>
                 <mesh filename="package://arduinobot_description/meshes/right_finger.STL" scale="0.01 0.01 0.01"/>
             </geometry>
         </visual>
+        <collision>
+            <origin xyz="-0.1 0.50 -0.1" rpy="0 0 -${PI/2}"/>
+            <geometry>
+                <mesh filename="package://arduinobot_description/meshes/right_finger.STL" scale="0.01 0.01 0.01"/>
+            </geometry>
+        </collision>
     </link>
-    <joint name="joint_4" type="revolute">
-        <parent link="claw_support" />
-        <child link="gripper_right" />
-        <axis xyz="0 0 1"/>
-        <origin rpy="0 0 0" xyz="-0.04 0.13 -0.1" />
-        <limit lower="-${PI/2}" upper="0.0" effort="${effort}" velocity="${velocity}"/>
-    </joint>
     <link name="gripper_left">
+        <xacro:default_inertial mass="0.01"/>
         <visual>
-                <origin rpy="0 0 -${PI/2}" xyz="-0.04 0.5 -0.1"/>
+            <origin xyz="-0.04 0.50 -0.1" rpy="0 0 -${PI/2}"/>
             <geometry>
                 <mesh filename="package://arduinobot_description/meshes/left_finger.STL" scale="0.01 0.01 0.01"/>
             </geometry>
         </visual>
+        <collision>
+            <origin xyz="-0.04 0.50 -0.1" rpy="0 0 -${PI/2}"/>
+            <geometry>
+                <mesh filename="package://arduinobot_description/meshes/left_finger.STL" scale="0.01 0.01 0.01"/>
+            </geometry>
+        </collision>
     </link>
-    <joint name="joint_5" type="revolute">
-        <parent link="claw_support" />
-        <child link="gripper_left" />
-        <axis xyz="0 0 1"/>
-        <origin rpy="0 0 0" xyz="-0.22 0.13 -0.1" />
-        <limit lower="0.0" upper="${PI/2}" effort="${effort}" velocity="${velocity}"/>
-        <mimic joint="joint_4" multiplier="-1"/>
-    </joint>
-    <link name="rgb_camera">
+    <!-- <link name="rgb_camera">
         <visual>
-            <origin rpy="-${PI/2} 0 -${PI/2}" xyz="-0.07 0.12 0.12" />
+            <origin xyz="-0.07 0.12 0.12" rpy="-${PI/2} 0 -${PI/2}"/>
             <geometry>
                 <mesh filename="package://arduinobot_description/meshes/pi_camera.STL" scale="0.01 0.01 0.01"/>
             </geometry>
         </visual>
-    </link>
-    <joint name="rgb_camera_joint" type="fixed">
+    </link> -->
+    <!-- Joints -->
+    <joint name="virtual_joint" type="fixed">
+        <origin xyz="0 0 0" rpy="0 0 0"/>
+        <parent link="world"/>
+        <child link="base_link"/>
+    </joint>
+    <joint name ="joint_1" type="revolute">
+        <origin xyz="0 0 0.307"/>
+        <parent link="base_link"/>
+        <child link = "base_plate"/>
+        <axis xyz="0 0 1"/>
+        <limit lower="-${PI / 2}" upper="${PI / 2}"
+               effort="${effort}" velocity="${velocity}"/>
+    </joint>
+    <joint name ="joint_2" type="revolute">
+        <origin xyz="-0.02 0 0.35"/>
+        <parent link="base_plate"/>
+        <child link = "forward_drive_arm"/>
+        <axis xyz="1 0 0"/>
+        <limit lower="-${PI / 2}" upper="${PI / 2}"
+                effort="${effort}" velocity="${velocity}"/>
+    </joint>
+    <joint name ="joint_3" type="revolute">
+        <origin xyz="0 0 0.8"/>
+        <parent link="forward_drive_arm"/>
+        <child link = "horizontal_arm"/>
+        <axis xyz="1 0 0"/>
+        <limit lower="-${PI / 2}" upper="${PI / 2}"
+               effort="${effort}" velocity="${velocity}"/>
+    </joint>
+    <joint name ="horizontal_arm_to_claw_support" type="fixed">
+        <origin xyz="0 0.82 0"/>
+        <parent link="horizontal_arm"/>
+        <child link = "claw_support"/>
+    </joint>
+    <joint name ="joint_4" type="revolute">
+        <origin xyz="-0.04 0.13 -0.1"/>
+        <parent link="claw_support"/>
+        <child link = "gripper_right"/>
+        <axis xyz="0 0 1"/>
+        <limit lower="-${PI / 2}" upper="0.0"
+               effort="${effort}" velocity="${velocity}"/>
+    </joint>
+    <joint name ="joint_5" type="revolute">
+        <origin xyz="-0.22 0.13 -0.1"/>
+        <parent link="claw_support"/>
+        <child link = "gripper_left"/>
+        <axis xyz="0 0 1"/>
+        <limit lower="0.0" upper="${PI / 2}"
+               effort="${effort}" velocity="${velocity}"/>
+        <mimic joint="joint_4" multiplier="-1"/>
+    </joint>
+    <!-- <joint name="rgb_camera_joint" type="fixed">
         <parent link="base_link" />
         <child link="rgb_camera" />
         <axis xyz="0 0 0"/>
-        <origin rpy="0 -0.5 1.57" xyz="0 0.45 0.2"/>
-    </joint>
+        <origin xyz="0 0.45 0.2" rpy="0 -0.5 1.57"/>
+    </joint> -->
 </robot>

Commit message: feat: :sparkles: Custom World for Gazebo to pre-change Physics step size

File: arduinobot_ws/src/arduinobot_description/urdf/arduinobot.urdf.xacro (robot description, xacro)
@@ -122,5 +122,5 @@
         </collision>
     </link>
-    <!-- <link name="rgb_camera">
+    <link name="rgb_camera">
         <visual>
             <origin xyz="-0.07 0.12 0.12" rpy="-${PI/2} 0 -${PI/2}"/>
@@ -129,5 +129,5 @@
             </geometry>
         </visual>
-    </link> -->
+    </link>
     <!-- Joints -->
     <joint name="virtual_joint" type="fixed">
@@ -182,9 +182,9 @@
         <mimic joint="joint_4" multiplier="-1"/>
     </joint>
-    <!-- <joint name="rgb_camera_joint" type="fixed">
+    <joint name="rgb_camera_joint" type="fixed">
         <parent link="base_link" />
         <child link="rgb_camera" />
         <axis xyz="0 0 0"/>
         <origin xyz="0 0.45 0.2" rpy="0 -0.5 1.57"/>
-    </joint> -->
+    </joint>
 </robot>

Commit message: feat: :sparkles: URDF and launch file modified for camera integration with plugins

File: arduinobot_ws/src/arduinobot_description/urdf/arduinobot.urdf.xacro (robot description, xacro)
@@ -1,4 +1,6 @@
 <?xml version="1.0"?>
 <robot xmlns:xacro="http://www.ros.org/wiki/xacro" name="arduinobot">
+    <!-- Include Gazebo Parameters -->
+    <xacro:include filename="$(find arduinobot_description)/urdf/arduinobot_gazebo.xacro" />
     <!-- Useful XACRO Variables (Properties) -->
     <xacro:property name="PI" value="3.14159265359" />
@@ -123,4 +125,5 @@
     </link>
     <link name="rgb_camera">
+        <xacro:default_inertial mass="0.001"/>
         <visual>
             <origin xyz="-0.07 0.12 0.12" rpy="-${PI/2} 0 -${PI/2}"/>
@@ -129,4 +132,10 @@
             </geometry>
         </visual>
+        <collision>
+            <origin xyz="-0.07 0.12 0.12" rpy="-${PI/2} 0 -${PI/2}"/>
+            <geometry>
+                <mesh filename="package://arduinobot_description/meshes/pi_camera.STL" scale="0.01 0.01 0.01"/>
+            </geometry>
+        </collision>
     </link>
     <!-- Joints -->
